File: mezzanine-0p5x1/mezzanine-0p5x1.kicad_sch (KiCad schematic)
At the start: 2 parts

Commit message: create test p5x1
Connections:
- net GND: now also U1.14 (GND), U1.23 (GND), U1.3 (GND), U1.33 (GND), U1.42 (GND), U1.51 (GND), U1.61 (GND)
- net an_0: now also U1.29 (an_0)
- net an_1: now also U1.30 (an_1)
- net an_2: now also U1.31 (an_2)
- net an_3: now also U1.34 (an_3)
- net bidir_0: now also U1.1 (bidir_0)
- net bidir_1: now also U1.2 (bidir_1)
- net bidir_2: now also U1.5 (bidir_2)
- net bidir_3: now also U1.6 (bidir_3)
- net bidir_34: now also U1.53 (bidir_34)
- net bidir_35: now also U1.54 (bidir_35)
- net bidir_36: now also U1.55 (bidir_36)
- net bidir_37: now also U1.56 (bidir_37)
- net bidir_38: now also U1.57 (bidir_38)
- net bidir_39: now also U1.58 (bidir_39)
- net bidir_4: now also U1.7 (bidir_4)
- net bidir_40: now also U1.59 (bidir_40)
- net bidir_41: now also U1.62 (bidir_41)
- net bidir_42: now also U1.63 (bidir_42)
- net bidir_43: now also U1.64 (bidir_43)
- net bidir_5: now also U1.8 (bidir_5)
- net clk: now also U1.65 (clk)
- net in_0: now also U1.67 (in_0)
- net in_1: now also U1.70 (in_1)
- net in_2: now also U1.71 (in_2)
- net in_3: now also U1.72 (in_3)
- net rst_n: now also U1.66 (rst_n)
