File: mezzanine-1x0p5/panelized/panel.kicad_pcb (KiCad board)
At the start: 4 copper layers, 77 x 82 mm, 220 parts

Commit message: remove two inner layers on panel
Other:
- copper layers 4 -> 2
Changed lines of the file:
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@@
 	(generator_version "10.0")
 	(general
-		(thickness 1.6)
+		(thickness 0.747)
 		(legacy_teardrops no)
 	)
@@
 	(layers
 		(0 "F.Cu" signal)
-		(4 "In1.Cu" signal)
-		(6 "In2.Cu" signal)
 		(2 "B.Cu" signal)
 		(9 "F.Adhes" user "F.Adhesive")
@@
 			)
 			(layer "dielectric 1"
-				(type "prepreg")
-				(thickness 0.196)
-				(material "FR4")
-				(epsilon_r 4.5)
-				(loss_tangent 0.02)
-			)
-			(layer "In1.Cu"
-				(type "copper")
-				(thickness 0.035)
-			)
-			(layer "dielectric 2"
 				(type "core")
-				(thickness 0.23)
-				(material "FR4")
-				(epsilon_r 4.5)
-				(loss_tangent 0.02)
-			)
-			(layer "In2.Cu"
-				(type "copper")
-				(thickness 0.035)
-			)
-			(layer "dielectric 3"
-				(type "prepreg")
-				(thickness 0.196)
+				(thickness 0.692)
 				(material "FR4")
 				(epsilon_r 4.5)
@@
 		(capping no)
 		(filling no)
+		(zone_defaults)
 		(aux_axis_origin 63.82 50.39)
 		(grid_origin 193.82 70.39)
